Commit message: 更改urdf文件 增加技术文档

File: urdf/aimibot.urdf (robot description, URDF)
Before this commit: robot aimibot, 10 links, 9 joints
Joints:
- joint realsense_joint: origin xyz=0.22476 -0.5145 4.8928E-05 rpy=1.5708 0 0 -> xyz=0.22476 4.8928E-05 0.5145  rpy=0 0 0; parent base_link -> base_footprint
